File: electronics/rpi-pico_to_arduino-nano/rpi-pico_to_arduino-nano.kicad_sch (KiCad schematic)
At the start: 41 parts, among them U1 Pico

Commit message: default closed solder jumpers, datasheets, erc
Parts:
- removed JP23_0, JP24_0, JP25_0, JP26_0, JP27_0, JP27_1: SolderJumper_2_Open, Jumper:SolderJumper-2_P1.3mm_Open_RoundedPad1.0x1.5mm, symbol Jumper:SolderJumper_2_Open
- added JP23_0, JP24_0, JP25_0, JP26_0, JP27_0, JP27_1: SolderJumper_2_Bridged, Jumper:SolderJumper-2_P1.3mm_Bridged_RoundedPad1.0x1.5mm, symbol Jumper:SolderJumper_2_Bridged
Connections:
- net +5V: now also JP25_0.1 (A)
- net 3V3: now also JP24_0.1 (A)
- net 3V3_pico: now also JP24_0.2 (B)
- net AGND: now also JP27_1.2 (B)
- net GND: now also JP27_0.1 (A), JP27_1.1 (A)
- net GND_pico: now also JP27_0.2 (B)
- net RUN: now also JP23_0.2 (B)
- net VBUS: now also JP25_0.2 (B)
- net VIN: now also JP26_0.1 (A)
- net VSYS: now also JP26_0.2 (B)
- net ~{RESET}: now also JP23_0.1 (A)
- net DO/RX renamed D0/RX
Other:
- note added: "Note: On Arduino Nano 33 BLE the pin AREF is present but not connected. (error in documentation)"
- note removed: "!!! TODO: check if connections at the Arduino make sense (done)=> Does the buzzer need an output with PWM? => yes and done => how does the rgb led work and with only one pin? => prüfen ob beim Arduino Nano 33 BLE AREF wirklich nirgends hin führt wenn ja: im Schema als Hinweis vermerken => entscheiden welche Lötjumper per default geschlossen sein sollen !!! Delete this text before when done"

Commit message: route pcb
Connections:
- net ~{RESET}: no longer A1.28 (~{RESET})
- no-connect marks 7 -> 8
Changed lines of the file:
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@@
 (kicad_sch (version 20211123) (generator eeschema)
   (paper "A4")
-  (junction (at 262.89 34.29) (diameter 0) (color 0 0 0 0)
-  )
   (junction (at 62.23 77.47) (diameter 0) (color 0 0 0 0)
   )
@@
   (junction (at 130.81 157.48) (diameter 0) (color 0 0 0 0)
   )
+  (no_connect (at 262.89 31.75))
   (no_connect (at 262.89 106.68))
   (no_connect (at 247.65 152.4))
@@
     (stroke (width 0) (type default) (color 0 0 0 0))
   )
-  (wire (pts (xy 262.89 31.75) (xy 262.89 34.29))
-    (stroke (width 0) (type default) (color 0 0 0 0))
-  )
   (wire (pts (xy 39.37 77.47) (xy 39.37 83.82))
     (stroke (width 0) (type default) (color 0 0 0 0))
@@
     (property "Reference" "U1" (id 0) (at 232.41 92.71 0))
     (property "Value" "Pico" (id 1) (at 232.41 95.25 0))
-    (property "Footprint" "MCU_RaspberryPi_and_Boards:RPi_Pico_SMD_TH" (id 2) (at 245.11 123.19 90)
-      (effects (font (size 1.27 1.27)) hide)
-    )
+    (property "Footprint" "MCU_RaspberryPi_and_Boards:RPi_Pico_SMD_TH" (id 2) (at 245.11 123.19 90))
     (property "Datasheet" "" (id 3) (at 245.11 123.19 0)
       (effects (font (size 1.27 1.27)) hide)

Commit message: add variables for workflow
Other:
- title: (none) -> rpi-pico_to_arduino-nano
Changed lines of the file:
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@@
 (kicad_sch (version 20211123) (generator eeschema)
   (paper "A4")
+  (title_block
+    (title "rpi-pico_to_arduino-nano")
+    (comment 1 "${PROJECT}")
+    (comment 2 "${PROJECT-URL}")
+    (comment 3 "${GIT-COMMIT-HASH}")
+    (comment 4 "${GIT-COMMIT-TAG}")
+  )
   (junction (at 62.23 77.47) (diameter 0) (color 0 0 0 0)
   )
