File: electronics/adapter/adapter.kicad_sch (KiCad schematic)
At the start: 41 parts, among them U1 Pico

Commit message: rename electronics project
Other:
- title: rpi-pico_to_arduino-nano -> Adapter
Changed lines of the file:
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@@
   (paper "A4")
   (title_block
-    (title "rpi-pico_to_arduino-nano")
+    (title "Adapter")
     (comment 1 "${PROJECT}")
     (comment 2 "${PROJECT-URL}")
